File: PCB-fuente_2step/PCB-fuente.kicad_pcb (KiCad board)
At the start: 2 copper layers, 146.7 x 80 mm, 19 parts, among them J1 ATX-20, J2 Limit_Switch 1, J3 Stepper 1, J4 Valvula, J5 Limit_Switch 2, J6 Board2Board_1, J7 Stepper 2, J8 Board2Board_2, Q1 2N7000, U1 DOIT_ESP32-DEVKIT, U2 IRFZ44N

Commit message: UPDATE 24-04-20 p2
Parts:
- R1, R2: moved to F.Cu
- moved C2 9.10 mm to (124.5, 68.9)
- moved J5 5.08 mm to (115.6, 86.4), turned to 270 degrees
- moved C1 1.27 mm to (121.9, 66.0), turned to 180 degrees
- moved R2 1.27 mm to (110.5, 76.5)
Routing:
- net -12V: track 0.00 -> 155.5 mm
- net +12V: track 57.3 -> 187.2 mm
- net +5V: track 148.2 -> 267.1 mm
- net -5V: track 0.00 -> 91.4 mm
- net +3V3: track 68.6 -> 130.5 mm
- net GND: track 35.8 -> 78.8 mm
- net I2C_SCL: track 143.4 -> 149.2 mm, vias 1 -> 0
- net Net-(J4-Pad2): track 20.8 -> 17.6 mm
- net Net-(Q1-Pad3): track 11.0 -> 9.72 mm
- net I2C_SDA: track 139.8 -> 138.7 mm, vias 1 -> 0
- added copper zone on B.Cu, net GND
Other:
- board size 146.7 x 80 mm -> 146.7 x 85.1 mm
