File: PCB-fuente_2step_ATmegaVF/PCB-fuente.kicad_pcb (KiCad board)
At the start: 2 copper layers, 127 x 95.2 mm, 55 parts, among them J1 ATX-20, J10 Ac_Ex_1, J11 Valvula, J12 Debug, J13 LimitSwitch3, J14 LimitSwitch4, J2 LimitSwitch1, J3 Stepper1, J4 Ac_Ex_2, J5 LimitSwitch2, J6 Board2Board_Sensors, J7 Stepper2, J8 Board2Board_Gui, J9 Power Redundancia, Q1 2N7000, Q2 2N7000, Q3 2N7000, Q4 2N7000, Q5 2N7000, U1 IRFZ44N, U2 IRFZ44N, U3 IRFZ44N, U4 74HC08, U5 74HC244

Commit message: NEW UPDATE 2-6-20
Parts:
- removed the REF** at (192.4, 60.3)
- removed the REF** at (192.4, 142.9)
- added REF**: MountingHole_2.5mm, MountingHole:MountingHole_2.5mm, F.Cu at (193.7, 64.1)
- added REF**: MountingHole_2.5mm, MountingHole:MountingHole_2.5mm, F.Cu at (193.7, 135.9)
- moved REF** 7.10 mm to (76.2, 135.9)
- moved REF** 4.02 mm to (76.2, 64.1)
Routing:
- net +5V: track 356.7 -> 354.8 mm
Other:
- board size 127 x 95.2 mm -> 126.4 x 81.9 mm

Commit message: UPDATE 11-6-20
Parts:
- added A1: Driver1_A4988, Module:Pololu_Breakout-16_15.2x20.3mm, F.Cu at (125.1, 33.7)
- added A1: Driver1_A4988, Module:Pololu_Breakout-16_15.2x20.3mm, F.Cu at (137.2, 128.9)
- added A2: Driver2_A4988, Module:Pololu_Breakout-16_15.2x20.3mm, F.Cu at (52.1, 34.3)
- added A2: Driver2_A4988, Module:Pololu_Breakout-16_15.2x20.3mm, F.Cu at (64.1, 129.5)
- added BZ1: Buzzer, Buzzer_Beeper:Buzzer_12x9.5RM7.6, F.Cu at (82.5, 22.9)
- added BZ1: Buzzer, Buzzer_Beeper:Buzzer_12x9.5RM7.6, F.Cu at (94.6, 118.1)
- added C1: 47uF, Capacitor_THT:CP_Radial_D5.0mm_P2.50mm, F.Cu at (82.5, 71.1)
- added C1: 47uF, Capacitor_THT:CP_Radial_D5.0mm_P2.50mm, F.Cu at (94.6, 166.4)
- added C2: 100nF, Capacitor_SMD:C_0805_2012Metric, B.Cu at (81.9, 64.8)
- added C2: 100nF, Capacitor_SMD:C_0805_2012Metric, B.Cu at (94.0, 160.0)
- added C3: 100uF, Capacitor_THT:CP_Radial_D5.0mm_P2.50mm, F.Cu at (123.8, 26.7)
- added C3: 100uF, Capacitor_THT:CP_Radial_D5.0mm_P2.50mm, F.Cu at (135.9, 121.9)
- added C4: 100uF, Capacitor_THT:CP_Radial_D5.0mm_P2.50mm, F.Cu at (52.1, 24.8)
- added C4: 100uF, Capacitor_THT:CP_Radial_D5.0mm_P2.50mm, F.Cu at (64.1, 120.0)
- added J1: ATX-20, Connector_Molex:Molex_Mini-Fit_Jr_5566-20A_2x10_P4.20mm_Vertical, F.Cu at (27.3, 24.1)
- added J1: ATX-20, Connector_Molex:Molex_Mini-Fit_Jr_5566-20A_2x10_P4.20mm_Vertical, F.Cu at (39.4, 119.4)
- added J10: Ac_Ex_1, TerminalBlock:TerminalBlock_bornier-2_P5.08mm, F.Cu at (55.9, 92.7)
- added J10: Ac_Ex_1, TerminalBlock:TerminalBlock_bornier-2_P5.08mm, F.Cu at (67.9, 188.0)
- added J11: Valvula, TerminalBlock:TerminalBlock_bornier-2_P5.08mm, F.Cu at (31.8, 92.7)
- added J11: Valvula, TerminalBlock:TerminalBlock_bornier-2_P5.08mm, F.Cu at (43.8, 188.0)
- added J12: Debug, Connector_Pin:Pin_D1.3mm_L11.0mm, F.Cu at (81.3, 47.0)
- added J12: Debug, Connector_Pin:Pin_D1.3mm_L11.0mm, F.Cu at (93.3, 142.2)
- added J13: LimitSwitch3, Connector_Molex:Molex_KK-254_AE-6410-03A_1x03_P2.54mm_Vertical, F.Cu at (123.2, 79.4)
- added J13: LimitSwitch3, Connector_Molex:Molex_KK-254_AE-6410-03A_1x03_P2.54mm_Vertical, F.Cu at (135.3, 174.6)
- added J14: LimitSwitch4, Connector_Molex:Molex_KK-254_AE-6410-03A_1x03_P2.54mm_Vertical, F.Cu at (123.2, 89.5)
- added J14: LimitSwitch4, Connector_Molex:Molex_KK-254_AE-6410-03A_1x03_P2.54mm_Vertical, F.Cu at (135.3, 184.8)
- added J2: LimitSwitch1, Connector_Molex:Molex_KK-254_AE-6410-03A_1x03_P2.54mm_Vertical, F.Cu at (123.2, 59.1)
- added J2: LimitSwitch1, Connector_Molex:Molex_KK-254_AE-6410-03A_1x03_P2.54mm_Vertical, F.Cu at (135.3, 154.3)
- added J3: Stepper1, Connector_Molex:Molex_KK-254_AE-6410-04A_1x04_P2.54mm_Vertical, F.Cu at (120.0, 24.1)
- added J3: Stepper1, Connector_Molex:Molex_KK-254_AE-6410-04A_1x04_P2.54mm_Vertical, F.Cu at (132.1, 119.4)
- added J4: Ac_Ex_2, TerminalBlock:TerminalBlock_bornier-2_P5.08mm, F.Cu at (43.8, 92.7)
- added J4: Ac_Ex_2, TerminalBlock:TerminalBlock_bornier-2_P5.08mm, F.Cu at (55.9, 188.0)
- added J5: LimitSwitch2, Connector_Molex:Molex_KK-254_AE-6410-03A_1x03_P2.54mm_Vertical, F.Cu at (123.2, 69.2)
- added J5: LimitSwitch2, Connector_Molex:Molex_KK-254_AE-6410-03A_1x03_P2.54mm_Vertical, F.Cu at (135.3, 164.5)
- added J6: Board2Board_Sensors, Connector_PinSocket_2.54mm:PinSocket_2x04_P2.54mm_Vertical, F.Cu at (78.7, 94.6)
- added J6: Board2Board_Sensors, Connector_PinSocket_2.54mm:PinSocket_2x04_P2.54mm_Vertical, F.Cu at (90.8, 189.9)
- added J7: Stepper2, Connector_Molex:Molex_KK-254_AE-6410-04A_1x04_P2.54mm_Vertical, F.Cu at (47.0, 24.1)
- added J7: Stepper2, Connector_Molex:Molex_KK-254_AE-6410-04A_1x04_P2.54mm_Vertical, F.Cu at (59.1, 119.4)
- added J8: Board2Board_Gui, Connector_PinSocket_2.54mm:PinSocket_2x04_P2.54mm_Vertical, F.Cu at (60.3, 21.6)
- added J8: Board2Board_Gui, Connector_PinSocket_2.54mm:PinSocket_2x04_P2.54mm_Vertical, F.Cu at (72.4, 116.8)
- added J9: Power Redundancia, TerminalBlock:TerminalBlock_bornier-6_P5.08mm, F.Cu at (22.2, 68.6)
- added J9: Power Redundancia, TerminalBlock:TerminalBlock_bornier-6_P5.08mm, F.Cu at (34.3, 163.8)
- added Q1: 2N7000, Package_TO_SOT_THT:TO-92_Inline, F.Cu at (41.3, 64.1)
- added Q1: 2N7000, Package_TO_SOT_THT:TO-92_Inline, F.Cu at (53.3, 159.4)
- added Q2: 2N7000, Package_TO_SOT_THT:TO-92_Inline, F.Cu at (83.8, 41.9)
- added Q2: 2N7000, Package_TO_SOT_THT:TO-92_Inline, F.Cu at (95.9, 137.2)
- added Q3: 2N7000, Package_TO_SOT_THT:TO-92_Inline, F.Cu at (108.6, 55.2)
- added Q3: 2N7000, Package_TO_SOT_THT:TO-92_Inline, F.Cu at (120.7, 150.5)
- added Q4: 2N7000, Package_TO_SOT_THT:TO-92_Inline, F.Cu at (47.6, 64.1)
- added Q4: 2N7000, Package_TO_SOT_THT:TO-92_Inline, F.Cu at (59.7, 159.4)
- added Q5: 2N7000, Package_TO_SOT_THT:TO-92_Inline, F.Cu at (34.9, 64.1)
- added Q5: 2N7000, Package_TO_SOT_THT:TO-92_Inline, F.Cu at (47.0, 159.4)
- added R1: 1K, Resistor_SMD:R_0805_2012Metric, F.Cu at (42.5, 58.1)
- added R1: 1K, Resistor_SMD:R_0805_2012Metric, F.Cu at (54.6, 153.4)
- added R10: 1K, Resistor_SMD:R_0805_2012Metric, F.Cu at (48.9, 58.1)
- added R10: 1K, Resistor_SMD:R_0805_2012Metric, F.Cu at (61.0, 153.3)
- added R11: 1K, Resistor_SMD:R_0805_2012Metric, F.Cu at (36.2, 58.1)
- added R11: 1K, Resistor_SMD:R_0805_2012Metric, F.Cu at (48.3, 153.4)
- added R12: 1M, Resistor_SMD:R_0805_2012Metric, B.Cu at (37.5, 70.8)
- added R12: 1M, Resistor_SMD:R_0805_2012Metric, B.Cu at (49.5, 166.1)
- added R13: 2K2, Resistor_SMD:R_0805_2012Metric, F.Cu at (116.2, 92.1)
- added R13: 2K2, Resistor_SMD:R_0805_2012Metric, F.Cu at (128.3, 187.3)
- added R14: 3K3, Resistor_SMD:R_0805_2012Metric, F.Cu at (116.2, 89.5)
- added R14: 3K3, Resistor_SMD:R_0805_2012Metric, F.Cu at (128.3, 184.8)
- added R15: 2K2, Resistor_SMD:R_0805_2012Metric, B.Cu at (49.5, 40.9)
- added R15: 2K2, Resistor_SMD:R_0805_2012Metric, B.Cu at (61.6, 136.2)
- added R16: 2K2, Resistor_SMD:R_0805_2012Metric, B.Cu at (122.6, 40.3)
- added R16: 2K2, Resistor_SMD:R_0805_2012Metric, B.Cu at (134.6, 135.6)
- added R17: 1M, Resistor_SMD:R_0805_2012Metric, B.Cu at (58.1, 59.7)
- added R17: 1M, Resistor_SMD:R_0805_2012Metric, B.Cu at (70.2, 154.9)
- added R18: 1M, Resistor_SMD:R_0805_2012Metric, B.Cu at (58.1, 57.1)
- added R18: 1M, Resistor_SMD:R_0805_2012Metric, B.Cu at (70.2, 152.4)
- added R19: 1K, Resistor_SMD:R_0805_2012Metric, B.Cu at (95.9, 66.4)
- added R19: 1K, Resistor_SMD:R_0805_2012Metric, B.Cu at (108.0, 161.6)
- added R2: 1M, Resistor_SMD:R_0805_2012Metric, B.Cu at (43.8, 70.8)
- added R2: 1M, Resistor_SMD:R_0805_2012Metric, B.Cu at (55.9, 166.0)
- added R3: 2K2, Resistor_SMD:R_0805_2012Metric, F.Cu at (116.2, 61.6)
- added R3: 2K2, Resistor_SMD:R_0805_2012Metric, F.Cu at (128.3, 156.8)
- added R4: 2K2, Resistor_SMD:R_0805_2012Metric, F.Cu at (116.2, 71.8)
- added R4: 2K2, Resistor_SMD:R_0805_2012Metric, F.Cu at (128.3, 167.0)
- added R5: 3K3, Resistor_SMD:R_0805_2012Metric, F.Cu at (116.2, 59.1)
- added R5: 3K3, Resistor_SMD:R_0805_2012Metric, F.Cu at (128.3, 154.3)
- added R6: 3K3, Resistor_SMD:R_0805_2012Metric, F.Cu at (116.2, 69.2)
- added R6: 3K3, Resistor_SMD:R_0805_2012Metric, F.Cu at (128.3, 164.5)
- added R7: 2K2, Resistor_SMD:R_0805_2012Metric, F.Cu at (116.2, 81.9)
- added R7: 2K2, Resistor_SMD:R_0805_2012Metric, F.Cu at (128.3, 177.2)
- added R8: 3K3, Resistor_SMD:R_0805_2012Metric, F.Cu at (116.2, 79.4)
- added R8: 3K3, Resistor_SMD:R_0805_2012Metric, F.Cu at (128.3, 174.6)
- added R9: 1M, Resistor_SMD:R_0805_2012Metric, B.Cu at (50.2, 70.8)
- added R9: 1M, Resistor_SMD:R_0805_2012Metric, B.Cu at (62.2, 166.1)
- added REF**: MountingHole_2.5mm, MountingHole:MountingHole_2.5mm, F.Cu at (130.2, 94.0)
- added REF**: MountingHole_2.5mm, MountingHole:MountingHole_2.5mm, F.Cu at (130.2, 22.2)
- added REF**: MountingHole_2.5mm, MountingHole:MountingHole_2.5mm, F.Cu at (12.7, 22.2)
- added REF**: MountingHole_2.5mm, MountingHole:MountingHole_2.5mm, F.Cu at (12.7, 94.0)
- added REF**: MountingHole_2.5mm, MountingHole:MountingHole_2.5mm, F.Cu at (142.2, 189.2)
- added REF**: MountingHole_2.5mm, MountingHole:MountingHole_2.5mm, F.Cu at (142.2, 117.5)
- added REF**: MountingHole_2.5mm, MountingHole:MountingHole_2.5mm, F.Cu at (24.8, 117.5)
- added REF**: MountingHole_2.5mm, MountingHole:MountingHole_2.5mm, F.Cu at (24.8, 189.2)
- added U1: IRFZ44N, Package_TO_SOT_THT:TO-220F-3_Vertical, F.Cu at (61.0, 83.2)
- added U1: IRFZ44N, Package_TO_SOT_THT:TO-220F-3_Vertical, F.Cu at (73.0, 178.4)
- added U2: IRFZ44N, Package_TO_SOT_THT:TO-220F-3_Vertical, F.Cu at (48.9, 83.2)
- added U2: IRFZ44N, Package_TO_SOT_THT:TO-220F-3_Vertical, F.Cu at (61.0, 178.4)
- added U3: IRFZ44N, Package_TO_SOT_THT:TO-220F-3_Vertical, F.Cu at (36.8, 83.2)
- added U3: IRFZ44N, Package_TO_SOT_THT:TO-220F-3_Vertical, F.Cu at (48.9, 178.4)
- added U4: 74HC08, Package_DIP:DIP-14_W7.62mm_LongPads, F.Cu at (99.7, 67.9)
- added U4: 74HC08, Package_DIP:DIP-14_W7.62mm_LongPads, F.Cu at (111.8, 163.2)
- added U5: 74HC244, Package_DIP:DIP-20_W7.62mm_LongPads, F.Cu at (99.7, 46.4)
- added U5: 74HC244, Package_DIP:DIP-20_W7.62mm_LongPads, F.Cu at (111.8, 141.6)
- added XA1: Arduino_Pro_Mini_3V3, PCB-fuente_2step_ATmega:Arduino_Mini_Socket, F.Cu at (78.7, 43.2)
- added XA1: Arduino_Pro_Mini_3V3, PCB-fuente_2step_ATmega:Arduino_Mini_Socket, F.Cu at (90.8, 138.4)
- moved A1 78.8 mm to (255.3, 33.7)
- moved A2 78.8 mm to (182.2, 34.3)
- moved C2 78.8 mm to (212.1, 64.8)
- moved C3 78.8 mm to (254.0, 26.7)
- moved C4 78.8 mm to (182.2, 24.8)
- moved J10 78.8 mm to (186.1, 92.7)
- moved J11 78.8 mm to (161.9, 92.7)
- moved J12 78.8 mm to (211.5, 47.0)
- moved J13 78.8 mm to (253.4, 79.4)
- moved J14 78.8 mm to (253.4, 89.5)
- moved J2 78.8 mm to (253.4, 59.1)
- moved J3 78.8 mm to (250.2, 24.1)
- moved J4 78.8 mm to (174.0, 92.7)
- moved J5 78.8 mm to (253.4, 69.2)
- moved J7 78.8 mm to (177.2, 24.1)
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Routing:
- net (no net): track 0.00 -> 5277.3 mm, vias 0 -> 38
- net +5V: track 354.8 -> 384.4 mm, vias 2 -> 0
- net GND: track 457.7 -> 464.4 mm, vias 2 -> 4
- net Net-(Q3-Pad3): track 23.2 -> 21.3 mm
- net ValvulaG: track 57.9 -> 56.4 mm
- net +12V: track 220.1 -> 219.6 mm, vias 3 -> 2
- net Dir: track 110.6 -> 111.0 mm, vias 3 -> 2
- net +3V3: vias 3 -> 4
- net Step_M1: vias 1 -> 0
- added copper zone on B.Cu, net (none)
Other:
- board size 126.4 x 81.9 mm -> 256.5 x 177.2 mm
- board text added: "Cara Frontal"
